File: PiEmulator.kicad_sch (KiCad schematic)
At the start: 45 parts, among them J1 Conn_01x01, J2 Conn_01x01, J3 USB_C_Receptacle_USB2.0, U1 ADA3708, U3 BQ24090DGQ, U4 TPS61230DRCR

Commit message: added jst moved usb-c
Parts:
- added U5: XD-XH-2AW-G, easyeda2kicad:CONN-TH_2P-P2.50_XH-2AW, symbol easyeda2kicad:XD-XH-2AW-G
Connections:
- net +BATT: now also U5.1
- net GND: now also U5.2
Changed lines of the file:
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@@
   (junction (at 237.49 71.755) (diameter 0) (color 0 0 0 0)
   )
+  (junction (at 241.3 60.325) (diameter 0) (color 0 0 0 0)
+  )
   (junction (at 91.44 46.355) (diameter 0) (color 0 0 0 0)
   )
@@
   )
   (junction (at 110.49 162.56) (diameter 0) (color 0 0 0 0)
+  )
+  (junction (at 237.49 57.785) (diameter 0) (color 0 0 0 0)
   )
   (junction (at 36.83 165.1) (diameter 0) (color 0 0 0 0)
@@
     (stroke (width 0) (type default))
   )
+  (wire (pts (xy 241.3 60.325) (xy 248.285 60.325))
+    (stroke (width 0) (type default))
+  )
   (wire (pts (xy 243.84 47.625) (xy 241.3 47.625))
     (stroke (width 0) (type default))
@@
     (stroke (width 0) (type default))
   )
+  (wire (pts (xy 237.49 57.785) (xy 237.49 61.595))
+    (stroke (width 0) (type default))
+  )
   (wire (pts (xy 88.9 71.755) (xy 91.44 71.755))
     (stroke (width 0) (type default))
@@
     (stroke (width 0) (type default))
   )
+  (wire (pts (xy 237.49 57.785) (xy 248.285 57.785))
+    (stroke (width 0) (type default))
+  )
   (wire (pts (xy 88.9 69.215) (xy 94.615 69.215))
     (stroke (width 0) (type default))
@@
     (stroke (width 0) (type default))
   )
+  (wire (pts (xy 241.3 60.325) (xy 241.3 71.755))
+    (stroke (width 0) (type default))
+  )
   (wire (pts (xy 95.885 56.515) (xy 88.9 56.515))
     (stroke (width 0) (type default))
@@
     (stroke (width 0) (type default))
   )
-  (wire (pts (xy 237.49 40.64) (xy 237.49 61.595))
+  (wire (pts (xy 237.49 40.64) (xy 237.49 57.785))
     (stroke (width 0) (type default))
   )
@@
     (stroke (width 0) (type default))
   )
-  (wire (pts (xy 241.3 47.625) (xy 241.3 71.755))
+  (wire (pts (xy 241.3 47.625) (xy 241.3 60.325))
     (stroke (width 0) (type default))
   )
@@
         )
       )
+    )
+  )
+  (symbol (lib_id "easyeda2kicad:XD-XH-2AW-G") (at 253.365 59.055 0) (unit 1)
+    (in_bom yes) (on_board yes) (dnp no) (fields_autoplaced)
+    (property "Reference" "U5" (at 256.54 57.785 0)
+      (effects (font (size 1.27 1.27)) (justify left))
+    )
+    (property "Value" "XD-XH-2AW-G" (at 256.54 60.325 0)
+      (effects (font (size 1.27 1.27)) (justify left))
+    )
+    (property "Footprint" "easyeda2kicad:CONN-TH_2P-P2.50_XH-2AW" (at 253.365 67.945 0)
+      (effects (font (size 1.27 1.27)) hide)
+    )
+    (property "Datasheet" "" (at 253.365 59.055 0)
+      (effects (font (size 1.27 1.27)) hide)
+    )
+    (property "LCSC Part" "C17700961" (at 253.365 70.485 0)
+      (effects (font (size 1.27 1.27)) hide)
+    )
+    (pin "1")
+    (pin "2")
+    (instances
+      (project "PiEmulator"
+        (path "/57df2d17-e1a3-4125-a0e7-53b56f3ddd17"
+          (reference "U5") (unit 1)
+        )
+      )

Commit message: added gerbers
Parts:
- added SW2: SS-12D10L5, easyeda2kicad:SW-TH_SS-12D10L5, symbol easyeda2kicad:SS-12D10L5
Connections:
- net +5V: now also SW2.1; no longer C5.2, C6.2, C7.2, R6.1, R8.2, U4.3 (VOUT), U4.4 (VOUT)
- new net: C5.2, C6.2, C7.2, R6.1, R8.2, SW2.2, U4.3 (VOUT), U4.4 (VOUT)
- no-connect marks 27 -> 28
Other:
- moved on the sheet: C1, C2, D1, D2, J1, J2, R1, R2, R3, R4, R5, U3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

Commit message: manufacturing changes
Parts:
- R1: value 540 -> 1K
Changed lines of the file:
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@@
   (symbol (lib_id "Device:R") (at 180.34 45.72 0) (unit 1)
     (in_bom yes) (on_board yes) (dnp no) (fields_autoplaced)
-    (property "Reference" "R1" (at 182.245 44.45 0)
+    (property "Reference" "R1" (at 182.88 44.45 0)
       (effects (font (size 1.27 1.27)) (justify left))
     )
-    (property "Value" "540" (at 182.245 46.99 0)
+    (property "Value" "1K" (at 182.88 46.99 0)
       (effects (font (size 1.27 1.27)) (justify left))
     )
